File: Hardware/ZX_Distance_and_Gesture_Sensor.sch (EAGLE design)
At the start: 0 parts

Commit message: Created comm ports, LED drivers, and LED receiver in schematic
Parts:
- added C1, C3, C5: 0.1uF, SparkFun-Capacitors:0.1UF-25V(+80/-20%)(0603)
- added C2, C4, C6: 10nF, SparkFun-Capacitors:10NF/10000PF-50V-10%(0603)
- added D1, D2: SFH4641, SparkFun-LED:SFH4641
- added FRAME1: FRAME-LETTER, SparkFun-Aesthetics:FRAME-LETTER
- added JP1: (no value), SparkFun-Connectors:M06SIP
- added JP2: (no value), SparkFun-Connectors:M05PTH
- added JP3: (no value), SparkFun-Connectors:M03PTH
- added Q1: MMBT2222A, SparkFun-DiscreteSemi:TRANSISTOR_NPNMMBT2222A
- added Q2: MOSFET-NCHANNEL2N7002PW, SparkFun-DiscreteSemi:MOSFET-NCHANNEL2N7002PW
- added R1, R5, R7: 100k, SparkFun-Resistors:100KOHM1/10W1%(0603)
- added R2: 330K, SparkFun-Resistors:330KOHM1/10W1%(0603)0603
- added R3: 10, SparkFun-Resistors:10OHM1/10W5%0603SMD
- added R4: 1K, SparkFun-Resistors:1KOHM1/10W1%(0603)
- added R6, R8: 1, SparkFun-Resistors:1OHM1/10W1%(0603)
- added U$1: PIC16F1823-14PINTSSOP, SparkFun-DigitalIC:PIC16F1823-14PINTSSOP
- added U$2: MCP6291T-E/OT, SparkFun-AnalogIC:MCP6291T-E/OT
- added U$3, U$4: DMC2700UDM, SparkFun-DiscreteSemi:DMC2700UDM
- added U$7: TSOP57238TT1, SparkFun-Sensors:TSOP57238TT1
Connections:
- new net CARRIER: R4.1
- new net COMMON: C4.1, C6.1, D1.C, D2.C, Q1.C
- new net DACOUT: R1.1
- new net DATA_RDY: JP3.1
- new net EM1: U$3.G1
- new net EM2: U$4.G1
- new net GND: C1.2, C2.2, C3.2, C5.2, JP1.5, JP1.6, JP2.2, Q2.S, R2.2, U$2.V-, U$3.S1, U$4.S1
- new net I2C_SCL: JP3.2
- new net I2C_SDA: JP3.3
- new net ICSPCLK: JP2.4
- new net ICSPDAT: JP2.5
- new net MCLR: JP2.3
- new net N$1: C2.1, R1.2, R2.1, U$2.+IN
- new net N$11: R8.1, U$4.D2
- new net N$12: D2.A, R8.2
- new net N$2: Q1.E, R3.2, U$2.-IN
- new net N$3: Q1.B, U$2.OUT
- new net N$4: Q2.D, R3.1
- new net N$5: Q2.G, R4.2
- new net N$6: R6.1, U$3.D2
- new net N$7: D1.A, R6.2
- new net N$8: R5.1, U$3.D1, U$3.G2
- new net N$9: R7.1, U$4.D1, U$4.G2
- new net UART_RX: JP1.3
- new net UART_TX: JP1.2
- new net VCC: C1.1, C3.1, C4.2, C5.1, C6.2, JP1.4, JP2.1, R5.2, R7.2, U$2.V+, U$3.S2, U$4.S2
Other:
- note added: "FTDI Basic"
- note added: "I2C"
- note added: "ICSP"
- note added: "Shawn Hymel of SparkFun Electronics With XYZ Interactive Technologies"
- note added: "v01"
