File: Hardware/ZX_Distance_and_Gesture_Sensor_PTH.brd (EAGLE design)
At the start: 55.9 x 12.7 mm, 50 parts, among them Q1 MMBT2222A, Q2 MOSFET-NCHANNEL2N7002PW, U1 BRM-2508VERT

Commit message: Updated REFDES numbers. Changed to v04.
Parts:
- removed U$1: PIC16F1823-14PINTSSOP, SparkFun-DigitalIC:TSSOP14
- added U5: BRM-2508VERT, SparkFun-Sensors:BRM-2508_VERT
- C2: value 10nF -> DNP
- U1: value BRM-2508VERT -> PIC16F1823-14PINTSSOP; device SparkFun-Sensors:BRM-2508_VERT -> SparkFun-DigitalIC:TSSOP14
- moved U1 5.08 mm to (0.00, 0.00), flipped to the bottom, turned to 90 degrees
- renumbered U$2 to U2, U$3 to U3, U$4 to U4, U$7 to U6
Connections:
- net CARRIER: now also U1.8; no longer U$1.8
- net EM1: now also U1.3; no longer U$1.3
- net EM2: now also U1.2; no longer U$1.2
- net GND: now also U1.14, U5.2; no longer U$1.14, U1.2
- net I2C_ADDR: now also U1.7; no longer U$1.7
- net I2C_SCL: now also U1.10; no longer U$1.10
- net I2C_SDA: now also U1.9; no longer U$1.9
- net ICSPCLK/DATA_RDY: now also U1.12; no longer U$1.12
- net ICSPDAT/DACOUT: now also U1.13; no longer U$1.13
- net MCLR: now also U1.4; no longer U$1.4
- net RECEIVER: now also U1.11, U5.1; no longer U$1.11, U1.1
- net UART_RX: now also U1.6; no longer U$1.6
- net UART_TX: now also U1.5; no longer U$1.5
- net VCC: now also U1.1, U5.3; no longer U$1.1, U1.3
Other:
- board text added: "v04"
- board text removed: "v03"

Commit message: Updated U2, U5, R2. Changed to v05.
Parts:
- FRAME1: value FRAME-LETTER -> (none)
- R10, R11: value 4.7k -> 4.7K; device SparkFun-Resistors:0603 -> SparkFun-Resistors:0603-RES
- R2: value 330K -> 100k
- SJ1: value (none) -> JUMPER-PAD-3-NC_BY_PASTE; device SparkFun-Passives:SJ_3_PASTE1&2&3 -> SparkFun-Passives:PAD-JUMPER-3-NC_BY_PASTE_YES_SILK_FULL_BOX
- SJ2: value SOLDERJUMPERNO -> JUMPER-PAD-2-NOYES_SILK; device SparkFun-Passives:SJ_2S-NO -> SparkFun-Passives:PAD-JUMPER-2-NO_YES_SILK
- U2: value MCP6291T-E/OT -> MCP6021T-E/OT
- U5: value BRM-2508VERT -> BRM-2A18VERT
Connections:
- net EM1: now also U3.G1; no longer U3.1
- net EM2: now also U4.G1; no longer U4.1
- net GND: now also U3.S1, U4.S1; no longer U3.5, U4.5
- net N$11: now also U4.D2; no longer U4.4
- net N$6: now also U3.D2; no longer U3.4
- net N$8: now also U3.D1, U3.G2; no longer U3.3, U3.6
- net N$9: now also U4.D1, U4.G2; no longer U4.3, U4.6
- net VCC: now also U3.S2, U4.S2; no longer U3.2, U4.2
Other:
- board text added: "v05"
- board text removed: "v04"

Commit message: Changed version number. Moved 1 trace. Removed ground pour under part.
Routing:
- net VCC: track 95.1 -> 97.2 mm
Other:
- board text added: "BLK"
- board text added: "GRN"
- board text added: "RXI"
- board text added: "TXO"
- board text added: "v10"
- board text removed: "NC"
- board text removed: "RX"
- board text removed: "TX"
- board text removed: "v05"

Commit message: Changed to 1% 10 ohm resistor. Added Arduino I2C address to schematic.
Parts:
- removed LOGO2: OSHW-LOGOS, SparkFun-Aesthetics:OSHW-LOGO-S
Changed lines of the file:
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@@
 <setting verticaltext="up"/>
 </settings>
-<grid distance="0.001" unitdist="inch" unit="inch" style="dots" multiple="1" display="yes" altdistance="0.0001" altunitdist="inch" altunit="inch"/>
+<grid distance="0.05" unitdist="inch" unit="inch" style="dots" multiple="1" display="yes" altdistance="0.005" altunitdist="inch" altunit="inch"/>
 <layers>
-<layer number="1" name="Top" color="4" fill="1" visible="yes" active="yes"/>
+<layer number="1" name="Top" color="4" fill="1" visible="no" active="yes"/>
 <layer number="2" name="Route2" color="1" fill="3" visible="no" active="yes"/>
 <layer number="15" name="Route15" color="4" fill="6" visible="no" active="yes"/>
-<layer number="16" name="Bottom" color="1" fill="1" visible="no" active="yes"/>
+<layer number="16" name="Bottom" color="1" fill="1" visible="yes" active="yes"/>
 <layer number="17" name="Pads" color="2" fill="1" visible="yes" active="yes"/>
 <layer number="18" name="Vias" color="2" fill="1" visible="yes" active="yes"/>
 <layer number="19" name="Unrouted" color="6" fill="1" visible="yes" active="yes"/>
 <layer number="20" name="Dimension" color="15" fill="1" visible="yes" active="yes"/>
-<layer number="21" name="tPlace" color="16" fill="1" visible="yes" active="yes"/>
-<layer number="22" name="bPlace" color="14" fill="1" visible="no" active="yes"/>
-<layer number="23" name="tOrigins" color="15" fill="1" visible="yes" active="yes"/>
-<layer number="24" name="bOrigins" color="15" fill="1" visible="no" active="yes"/>
+<layer number="21" name="tPlace" color="16" fill="1" visible="no" active="yes"/>
+<layer number="22" name="bPlace" color="14" fill="1" visible="yes" active="yes"/>
+<layer number="23" name="tOrigins" color="15" fill="1" visible="no" active="yes"/>
+<layer number="24" name="bOrigins" color="15" fill="1" visible="yes" active="yes"/>
 <layer number="25" name="tNames" color="7" fill="1" visible="no" active="yes"/>
 <layer number="26" name="bNames" color="7" fill="1" visible="no" active="yes"/>
@@
 <layer number="56" name="wert" color="7" fill="1" visible="no" active="no"/>
 <layer number="57" name="tCAD" color="7" fill="1" visible="no" active="no"/>
+<layer number="59" name="tCarbon" color="7" fill="1" visible="no" active="no"/>
+<layer number="60" name="bCarbon" color="7" fill="1" visible="no" active="no"/>
 <layer number="90" name="Modules" color="5" fill="1" visible="no" active="no"/>
 <layer number="91" name="Nets" color="2" fill="1" visible="no" active="no"/>
@@
 <layer number="127" name="_tValues" color="7" fill="1" visible="no" active="no"/>
 <layer number="128" name="_bValues" color="7" fill="1" visible="no" active="no"/>
+<layer number="129" name="Mask" color="7" fill="1" visible="no" active="yes"/>
 <layer number="131" name="tAdjust" color="7" fill="1" visible="no" active="no"/>
 <layer number="132" name="bAdjust" color="7" fill="1" visible="no" active="no"/>
@@
 <layer number="223" name="223bmp" color="24" fill="1" visible="no" active="no"/>
 <layer number="224" name="224bmp" color="25" fill="1" visible="no" active="no"/>
+<layer number="225" name="225bmp" color="7" fill="1" visible="no" active="yes"/>
+<layer number="226" name="226bmp" color="7" fill="1" visible="no" active="yes"/>
+<layer number="227" name="227bmp" color="7" fill="1" visible="no" active="yes"/>
+<layer number="228" name="228bmp" color="7" fill="1" visible="no" active="yes"/>
+<layer number="229" name="229bmp" color="7" fill="1" visible="no" active="yes"/>
+<layer number="230" name="230bmp" color="7" fill="1" visible="no" active="yes"/>
+<layer number="231" name="231bmp" color="7" fill="1" visible="no" active="yes"/>
 <layer number="248" name="Housing" color="7" fill="1" visible="no" active="no"/>
 <layer number="249" name="Edge" color="7" fill="1" visible="no" active="no"/>
@@
 <wire x1="14.4526" y1="-3.3528" x2="12.9794" y2="-3.3528" width="0.254" layer="42"/>
 <wire x1="12.9794" y1="-3.3528" x2="12.6492" y2="-3.683" width="0.254" layer="42"/>
+<text x="-10.16" y="-4.064" size="0.8128" layer="22" font="vector" ratio="15" rot="MR0" align="bottom-center">GRN</text>
+<text x="-7.62" y="-4.064" size="0.8128" layer="22" font="vector" ratio="15" rot="MR0" align="bottom-center">TXO</text>
+<text x="-5.08" y="-4.064" size="0.8128" layer="22" font="vector" ratio="15" rot="MR0" align="bottom-center">RXI</text>
+<text x="-2.54" y="-4.064" size="0.8128" layer="22" font="vector" ratio="15" rot="MR0" align="bottom-center">VCC</text>
+<text x="0" y="-4.064" size="0.8128" layer="22" font="vector" ratio="15" rot="MR0" align="bottom-center">GND</text>
+<text x="2.54" y="-4.064" size="0.8128" layer="22" font="vector" ratio="15" rot="MR0" align="bottom-center">BLK</text>
+<text x="5.08" y="-4.064" size="0.8128" layer="22" font="vector" ratio="15" rot="MR0" align="bottom-center">DR</text>
+<text x="7.62" y="-4.064" size="0.8128" layer="22" font="vector" ratio="15" rot="MR0" align="bottom-center">CL</text>
+<text x="10.16" y="-4.064" size="0.8128" layer="22" font="vector" ratio="15" rot="MR0" align="bottom-center">DA</text>
 </plain>
 <attributes>
@@
 </element>
 <element name="R3" library="SparkFun-Resistors" package="0603-RES" value="10" x="12.7" y="0" rot="MR270">
-<attribute name="PROD_ID" value="RES-09834" x="60.96" y="-22.86" size="1.778" layer="28" rot="MR270" display="off"/>
+<attribute name="PROD_ID" value="RES-12581" x="60.96" y="-22.86" size="1.778" layer="28" rot="MR270" display="off"/>
+<attribute name="TOL" value="1%" x="12.7" y="0" size="1.778" layer="28" rot="MR270" display="off"/>
 </element>
 <element name="R4" library="SparkFun-Resistors" package="0603-RES" value="1K" x="6.35" y="1.27" rot="MR180">
@@
 <element name="U$5" library="SparkFun-Aesthetics" package="SFE_LOGO_NAME_FLAME_.1" value="SFE_LOGO_NAME_FLAME.1_INCH" x="3.7592" y="0.6604"/>
 <element name="LOGO1" library="SparkFun-Aesthetics" package="SFE_LOGO_FLAME_.1" value="SFE_LOGO_FLAME.1_INCH" x="-22.225" y="-5.08" rot="MR0"/>
-<element name="LOGO2" library="SparkFun-Aesthetics" package="OSHW-LOGO-S" value="OSHW-LOGOS" x="23.495" y="3.81" rot="MR0"/>
 <element name="STANDOFF1" library="SparkFun-Electromechanical" package="STAND-OFF" value="STAND-OFF" x="-25.4" y="0"/>
 <element name="STANDOFF2" library="SparkFun-Electromechanical" package="STAND-OFF" value="STAND-OFF" x="25.4" y="0"/>
