File: Production_Files/ZX_Distance_and_Gesture_Sensor_PTH_Panel_v10.brd (EAGLE design)
At the start: 132.1 x 145.3 mm, 963 parts, among them Q1 MMBT2222A, Q10 MOSFET-NCHANNEL2N7002PW, Q11 MMBT2222A, Q12 MOSFET-NCHANNEL2N7002PW, Q13 MMBT2222A, Q14 MOSFET-NCHANNEL2N7002PW, Q15 MMBT2222A, Q16 MOSFET-NCHANNEL2N7002PW, Q17 MMBT2222A, Q18 MOSFET-NCHANNEL2N7002PW, Q19 MMBT2222A, Q2 MOSFET-NCHANNEL2N7002PW, Q20 MOSFET-NCHANNEL2N7002PW, Q21 MMBT2222A, Q22 MOSFET-NCHANNEL2N7002PW, Q23 MMBT2222A, Q24 MOSFET-NCHANNEL2N7002PW, Q25 MMBT2222A, Q26 MOSFET-NCHANNEL2N7002PW, Q27 MMBT2222A, Q28 MOSFET-NCHANNEL2N7002PW, Q29 MMBT2222A, Q3 MMBT2222A, Q30 MOSFET-NCHANNEL2N7002PW, Q31 MMBT2222A, Q32 MOSFET-NCHANNEL2N7002PW, Q33 MMBT2222A, Q34 MOSFET-NCHANNEL2N7002PW, Q35 MMBT2222A, Q36 MOSFET-NCHANNEL2N7002PW, Q37 MMBT2222A, Q38 MOSFET-NCHANNEL2N7002PW, Q39 MMBT2222A, Q4 MOSFET-NCHANNEL2N7002PW, Q40 MOSFET-NCHANNEL2N7002PW, Q5 MMBT2222A, Q6 MOSFET-NCHANNEL2N7002PW, Q7 MMBT2222A, Q8 MOSFET-NCHANNEL2N7002PW, Q9 MMBT2222A, U1 PIC16F1823-14PINTSSOP, U10 DMC2700UDM, U100 DMC2700UDM, U101 TSOP57238TT1, U102 BRM-2A18VERT, U103 PIC16F1823-14PINTSSOP, U104 MCP6021T-E/OT, U105 DMC2700UDM, U106 DMC2700UDM, U107 TSOP57238TT1, U108 BRM-2A18VERT, U109 PIC16F1823-14PINTSSOP, U11 TSOP57238TT1, U110 MCP6021T-E/OT, U111 DMC2700UDM, U112 DMC2700UDM, U113 TSOP57238TT1, U114 BRM-2A18VERT, U115 PIC16F1823-14PINTSSOP, U116 MCP6021T-E/OT, U117 DMC2700UDM, U118 DMC2700UDM, U119 TSOP57238TT1, U12 BRM-2A18VERT, U120 BRM-2A18VERT, U13 PIC16F1823-14PINTSSOP, U14 MCP6021T-E/OT, U15 DMC2700UDM, U16 DMC2700UDM, U17 TSOP57238TT1, U18 BRM-2A18VERT, U19 PIC16F1823-14PINTSSOP, U2 MCP6021T-E/OT, U20 MCP6021T-E/OT, U21 DMC2700UDM, U22 DMC2700UDM, U23 TSOP57238TT1, U24 BRM-2A18VERT, U25 PIC16F1823-14PINTSSOP, U26 MCP6021T-E/OT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

Commit message: added bottom side panel fiducials
Parts:
- added E$3: (no value), SparkFun-Retired:FIDUCIAL-1.5X3
- added E$4, E$6: (no value), SparkFun-Aesthetics:FIDUCIAL-1X2
Changed lines of the file:
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@@
 <?xml version="1.0" encoding="utf-8"?>
 <!DOCTYPE eagle SYSTEM "eagle.dtd">
-<eagle version="6.6.0">
+<eagle version="7.2.0">
 <drawing>
 <settings>
@@
 <pass name="Default">
 <param name="RoutingGrid" value="50mil"/>
+<param name="AutoGrid" value="1"/>
+<param name="Efforts" value="0"/>
+<param name="TopRouterVariant" value="1"/>
 <param name="tpViaShape" value="round"/>
 <param name="PrefDir.1" value="|"/>
@@
 <element name="E$5" library="SparkFun-Aesthetics" package="FIDUCIAL-1X2" value="" x="127.635" y="132.588" rot="R180"/>
 <element name="E$1" library="SparkFun-Retired" package="FIDUCIAL-1.5X3" value="" x="4.572" y="13.208"/>
+<element name="E$3" library="SparkFun-Retired" package="FIDUCIAL-1.5X3" value="" x="4.572" y="13.208" rot="MR0"/>
+<element name="E$4" library="SparkFun-Aesthetics" package="FIDUCIAL-1X2" value="" x="127.635" y="11.938" rot="MR0"/>
+<element name="E$6" library="SparkFun-Aesthetics" package="FIDUCIAL-1X2" value="" x="127.635" y="132.588" rot="MR180"/>
 </elements>
 <signals>
